File: LoLin32-Lora.brd (EAGLE design)
At the start: 51.1 x 25.7 mm, 27 parts, among them J4 1X2-3.5MM, Q1 BSS138, U1 24AA02E64T

Commit message: Bump to V1.1
Parts:
- removed J4: 1X2-3.5MM, adafruit:1X2-3.5MM
- removed OK1: LVT814, optocoupler:DIL4-SMD
- removed Q1: BSS138, Seeed-Discrete:SOT23
- removed R3: 1.5K, _c2h:0805-RES
- removed R4, R6: 10k, _c2h:0805-RES
- added JRF, JRN: (no value), SparkFun-Passives:PAD-JUMPER-2-NO_NO_SILK
- added U$1: RN2483, _c2h:RN2483_NOGPIO_868
- moved U$4 22.9 mm to (34.7, 34.0)
- moved U$6 11.3 mm to (26.0, 26.8), turned to 90 degrees
- moved GROVE_I2C 10.2 mm to (12.7, 29.8)
- moved I2C_OLED 10.2 mm to (17.4, 29.8)
- moved R1 10.2 mm to (26.7, 33.5)
- moved R2 10.2 mm to (26.7, 36.6)
- moved U$2 10.2 mm to (22.2, 27.3)
- moved U$3 10.2 mm to (22.2, 32.4)
- moved C2 4.15 mm to (42.0, 33.7), turned to 270 degrees
- moved U$5 3.81 mm to (38.1, 29.8)
- moved U1 1.42 mm to (16.0, 36.8)
- moved C1 0.99 mm to (11.2, 37.1), flipped to the bottom, turned to 0 degrees
Connections:
- removed net ANT: J$2.ANT1, J$2.ANT2, J$2.ANT3, U$5.ANT
- removed net N$8: OK1.3, Q1.1, R4.2
- net 3V3: now also U$1.VDD, U$1.VDD2; no longer R6.2
- net GND: now also U$1.GND, U$1.GND11, U$1.GND12, U$1.GND3, U$1.GND4, U$1.GND7, U$1.GND9; no longer Q1.2, R4.1
- net IO16: no longer Q1.3, R6.1
- net IO25: now also U$1.UART_RX, U$5.RST; no longer U$5.DIO5
- net IO34: no longer OK1.4
- net IO35: now also U$1.UART_TX, U$5.DIO5; no longer U$5.RST
- net IO4: now also U$1.RESET°
- net N$5: now also JRN.2, U$1.RFH; no longer J4.2, OK1.2
- net N$6: now also JRF.1, U$5.ANT; no longer J4.1, R3.1
- net N$7: now also J$2.ANT1, J$2.ANT2, J$2.ANT3, JRF.2, JRN.1; no longer OK1.1, R3.2
Routing:
- net IO16: track 38.7 -> 0.00 mm
- net 3V3: track 56.5 -> 73.7 mm, vias 1 -> 2
- net SDA: track 45.2 -> 30.3 mm
- net IO34: track 13.6 -> 0.00 mm
- net IO13: track 23.2 -> 35.0 mm, vias 0 -> 1
- net SCL: track 36.5 -> 26.5 mm
- net 5V: track 23.5 -> 32.1 mm
- net IO4: track 4.46 -> 11.9 mm
- net N$8: track 6.74 -> 0.00 mm
- net ANT: track 5.48 -> 0.00 mm
- net N$5: track 9.72 -> 5.16 mm
- net IO18: track 13.1 -> 16.9 mm
- net N$7: track 10.7 -> 7.19 mm
- net IO25: track 10.5 -> 13.3 mm
- net IO5: track 16.9 -> 19.4 mm
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Other:
- board text added: "24AA"
- board text added: "Lora"
- board text added: "Node32"
- board text added: "V1.1"
- board text removed: "24AA02"
- board text removed: "Teleinfo"
- board text removed: "V1.0"
