File: LoLin32-Lora.sch (EAGLE design)
At the start: 25 parts, among them J4 1X2-3.5MM, Q1 BSS138, U1 24AA02E64T

Commit message: Bump to V1.1
Parts:
- removed J4: 1X2-3.5MM, adafruit:1X2-3.5MM
- removed OK1: LVT814, optocoupler:SFH6206
- removed Q1: BSS138, Seeed-Discrete:MOSFET-N-''
- removed R3: 1.5K, _c2h:RESISTOR0805-RES
- removed R4, R6: 10k, _c2h:RESISTOR0805-RES
- added JRF, JRN: JUMPER-PAD-2-NO, SparkFun-Passives:JUMPER-PAD-2-NO
- added U$1: RN2483, _c2h:RN2483_NOGPIO868
Connections:
- removed net ANT: J$2.SIGNAL, U$5.ANT
- removed net N$8: OK1.E, Q1.G, R4.2
- net 3V3: now also U$1.VDD; no longer R6.2
- net GND: now also U$1.GND; no longer Q1.S, R4.1
- net IO16: no longer Q1.D, R6.1
- net IO25: now also U$1.RX, U$5.RST; no longer U$5.DIO5
- net IO34: no longer OK1.C
- net IO35: now also U$1.TX, U$5.DIO5; no longer U$5.RST
- net IO4: now also U$1.RESET°
- net N$5: now also JRN.2, U$1.RFH; no longer J4.2, OK1.AC2
- net N$6: now also JRF.1, U$5.ANT; no longer J4.1, R3.1
- net N$7: now also J$2.SIGNAL, JRF.2, JRN.1; no longer OK1.AC1, R3.2
Other:
- note added: "BUILT_IN LED"
- note removed: "J1"
- note removed: "Téléinfo"
- note removed: "WeMos has a 12K pulldown on GPIO15"
- moved on the sheet: J1, J2, J3
